File: design/MicroUSB2DIP.kicad_pcb (KiCad board)
At the start: 2 copper layers, 15 x 13.4 mm, 4 parts, among them J1 UJ2-MIBH-G-SMT-TR, J2 TS-101-X-A-1, J3 TS-101-X-A-1, J4 TS-105-T-A-1

Commit message: pictures edit
Other:
- board text added: "D+"
- board text added: "D-"
- board text added: "GND"
- board text added: "IO"
- board text added: "VBUS"
Changed lines of the file:
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@@
 		(at 64.3 57.5 -90)
 		(property "Reference" "J4"
-			(at -5.9 2.3 0)
+			(at -1.35 3.2 0)
 			(layer "F.SilkS")
 			(effects
@@
 		)
 	)
+	(gr_text "D-"
+		(at 62.6 55 90)
+		(layer "Cmts.User")
+		(effects
+			(font
+				(size 0.5 0.5)
+				(thickness 0.125)
+			)
+		)
+	)
+	(gr_text "D+\n"
+		(at 62.6 57.4 90)
+		(layer "Cmts.User")
+		(effects
+			(font
+				(size 0.5 0.5)
+				(thickness 0.125)
+			)
+		)
+	)
+	(gr_text "GND"
+		(at 62.6 62.6 90)
+		(layer "Cmts.User")
+		(effects
+			(font
+				(size 0.5 0.5)
+				(thickness 0.125)
+			)
+		)
+	)
+	(gr_text "IO"
+		(at 62.6 60 90)
+		(layer "Cmts.User")
+		(effects
+			(font
+				(size 0.5 0.5)
+				(thickness 0.125)
+			)
+		)
+	)
+	(gr_text "VBUS"
+		(at 62.6 52.4 90)
+		(layer "Cmts.User")
+		(effects
+			(font
+				(size 0.5 0.5)
+				(thickness 0.125)
+			)
+		)
+	)
 	(dimension
 		(type aligned)
@@
 			(xy 60.1 53.2) (xy 60.93 51.86)
 		)
-		(leader_length 6.930978)
+		(leader_length 6.386998)
 		(gr_text "D=3 mm"
-			(at 71.711657 45.967768 0)
+			(at 71.425212 46.430222 0)
 			(layer "Cmts.User")
 			(effects
